Commit message: Fixed files for ridgeback_intel_description

File: ridgeback_description/urdf/ridgeback.urdf.xacro (robot description, xacro)
@@ -264,187 +264,4 @@
     <origin xyz="0 0 ${deck_height}" rpy="0 0 0"/>
   </joint>
-  <!-- Constants for camera mount  dimensions -->
-<xacro:property name="massp" value="0.05" /> <!-- arbitrary value for mass -->
-   <xacro:property name="widthp" value="0.025" /> <!-- Radius of the camera mount -->
-   <xacro:property name="heightp" value="0.085" /> <!--Height of the camera mount -->
-   <xacro:property name="mass" value="0.05" /> <!-- arbitrary value for mass -->
-   <xacro:property name="width" value="0.02" /> <!-- Radius of the camera mount -->
-   <xacro:property name="height" value="0.085" /> <!--Height of the camera mount -->
-   <xacro:property name="camera_length" value="0.0492" /> <!-- Size of square 'camera' box -->
-   <xacro:property name="camera_width" value="0.025" /> <!-- Space btw top of beam and the each joint -->
-   <xacro:property name="angle_diff" value="${pi/3}" /> <!-- Space btw top of beam and the each joint -->
-   <xacro:property name="angle_tilt_1" value="0" /> <!-- Space btw top of beam and the each joint -->
-   <xacro:property name="angle_tilt_2" value="0" /> <!-- Space btw top of beam and the each joint -->
-   <xacro:property name="angle_tilt_3" value="0" /> <!-- Space btw top of beam and the each joint -->
-   <!-- Import all Gazebo-customization elements, including Gazebo colors -->
-  <xacro:include filename="$(find ridgeback_description)/urdf/multi_d435.gazebo" />
-  <joint name="ridgeback_to_mount" type="fixed">
-    <parent link="base_link" />
-    <child link="mount_tripod" />
-    <origin rpy="0 0 0" xyz="0.215 0 1.21" />
-  </joint>
-   <!-- Tripod -->
-      <link name="mount_tripod">
-        <collision>
-          <origin xyz="0 0 ${heightp/2}" rpy="0 0 0"/>
-          <geometry>
-             <cylinder radius="${widthp}" length="${heightp}"/>
-          </geometry>
-        </collision>
-        <visual>
-          <origin xyz="0 0 0" rpy="${pi/2} 0 0"/>
-          <geometry>
-    	       <mesh filename="package://ridgeback_description/meshes/tripod_simplified.STL"/>
-          </geometry>
-          <material name="orange"/>
-        </visual>
-        <inertial>
-          <origin xyz="0 0 ${heightp/2}" rpy="0 0 0"/>
-          <mass value="${massp}"/>
-          <inertia
-    	  ixx="${massp / 12.0 * (widthp*widthp + heightp*heightp)}" ixy="0.0" ixz="0.0"
-    	  iyy="${massp / 12.0 * (heightp*heightp + widthp*widthp)}" iyz="0.0"
-    	  izz="${massp / 12.0 * (widthp*widthp + widthp*widthp)}"/>
-        </inertial>
-      </link>
-      <joint name="camera_mount_joint" type="fixed">
-        <parent link="mount_tripod" />
-        <child link="multi_d435_mount" />
-        <origin rpy="0 0 0" xyz="0 0 ${heightp} " />
-      </joint>
-      <!-- Camera mount Link -->
-      <link name="multi_d435_mount">
-        <collision>
-          <origin xyz="0 0 ${height/2}" rpy="0 0 0"/>
-          <geometry>
-             <cylinder radius="${width}" length="${height}"/>
-          </geometry>
-        </collision>
-       <visual>
-          <origin xyz="0 0 0" rpy="0 0 ${pi/6}"/>
-          <geometry>
-    	       <mesh filename="package://ridgeback_description/meshes/D435x6_mounting-support.STL"/>
-          </geometry>
-        </visual>
-        <inertial>
-          <origin xyz="0 0 ${height/2}" rpy="0 0 0"/>
-          <mass value="${mass}"/>
-          <inertia
-    	  ixx="${mass / 12.0 * (width*width + height*height)}" ixy="0.0" ixz="0.0"
-    	  iyy="${mass / 12.0 * (height*height + width*width)}" iyz="0.0"
-    	  izz="${mass / 12.0 * (width*width + width*width)}"/>
-        </inertial>
-      </link>
-      <joint name="camera_joint_1" type="fixed">
-        <origin xyz="${width+camera_width} 0 ${height-camera_length}" rpy="${pi/2} ${angle_tilt_1} 0"/>
-        <parent link="multi_d435_mount"/>
-        <child link="camera1_link"/>
-      </joint>
-      <joint name="camera_joint_2" type="fixed">
-        <origin xyz="${(width+camera_width)*cos(angle_diff)} ${(width+camera_width)*sin(angle_diff)} ${height-camera_length}" rpy="${pi/2} ${angle_tilt_2} ${angle_diff}"/>
-        <parent link="multi_d435_mount"/>
-        <child link="camera2_link"/>
-      </joint>
-      <joint name="camera_joint_3" type="fixed">
-        <origin xyz="${(width+camera_width)*cos(angle_diff)} -${(width+camera_width)*sin(angle_diff)} ${height-camera_length}" rpy="${pi/2} ${angle_tilt_3} -${angle_diff}"/>
-        <parent link="multi_d435_mount"/>
-        <child link="camera3_link"/>
-      </joint>
-      <!-- Camera 1-->
-      <link name="camera1_link">
-        <collision>
-          <origin xyz="0 0 0" rpy="0 0 0"/>
-          <geometry>
-    	       <box size="${camera_width} ${camera_length} ${camera_width}"/>
-          </geometry>
-        </collision>
-        <visual>
-          <origin xyz="0 0 0" rpy="${pi/2} 0 ${pi/2}"/>
-          <geometry>
-    	       <mesh filename="package://ridgeback_description/meshes/Intel_RealSense_Depth_Camera_D435.STL"/>
-          </geometry>
-          <material name="red"/>
-        </visual>
-        <inertial>
-          <mass value="0.0615752" />
-          <origin xyz="0 0 0" rpy="0 0 0"/>
-          <inertia ixx="9.108e-05" ixy="0" ixz="0" iyy="2.51e-06" iyz="0" izz="8.931e-05" />
-        </inertial>
-      </link>
-      <!-- Camera 2-->
-      <link name="camera2_link">
-        <collision>
-          <origin xyz="0 0 0" rpy="0 0 0"/>
-          <geometry>
-    	       <box size="${camera_length} ${camera_width} ${camera_width}"/>
-          </geometry>
-        </collision>
-        <visual>
-          <origin xyz="0 0 0" rpy="${pi/2} 0 ${pi/2}"/>
-          <geometry>
-    	       <mesh filename="package://ridgeback_description/meshes/Intel_RealSense_Depth_Camera_D435.STL"/>
-          </geometry>
-          <material name="red"/>
-        </visual>
-        <inertial>
-          <mass value="0.0615752" />
-          <origin xyz="0 0 0" rpy="0 0 0"/>
-          <inertia ixx="9.108e-05" ixy="0" ixz="0" iyy="2.51e-06" iyz="0" izz="8.931e-05" />
-        </inertial>
-      </link>
-      <!-- Camera 3-->
-      <link name="camera3_link">
-        <collision>
-          <origin xyz="0 0 0" rpy="0 0 0"/>
-          <geometry>
-    	       <box size="${camera_length} ${camera_width} ${camera_width}"/>
-          </geometry>
-        </collision>
-        <visual>
-          <origin xyz="0 0 0" rpy="${pi/2} 0 ${pi/2}"/>
-          <geometry>
-    	       <mesh filename="package://ridgeback_description/meshes/Intel_RealSense_Depth_Camera_D435.STL"/>
-          </geometry>
-          <material name="red"/>
-        </visual>
-        <inertial>
-          <mass value="0.0615752" />
-          <origin xyz="0 0 0" rpy="0 0 0"/>
-          <inertia ixx="9.108e-05" ixy="0" ixz="0" iyy="2.51e-06" iyz="0" izz="8.931e-05" />
-        </inertial>
-      </link>
-  <!-- generate an optical frame http://www.ros.org/reps/rep-0103.html#suffix-frames
-      so that ros and opencv can operate on the camera frame correctly -->
-    <joint name="camera_optical_joint_1" type="fixed">
-    <!-- these values have to be these values otherwise the gazebo camera image
-        won't be aligned properly with the frame it is supposedly originating from -->
-    <origin xyz="0 0 0" rpy="${-pi/2} 0 ${-pi/2}"/>
-    <parent link="camera1_link"/>
-    <child link="camera_link_optical_1"/>
-  </joint>
-  <link name="camera_link_optical_1">
-  </link>
-  <!-- generate an optical frame http://www.ros.org/reps/rep-0103.html#suffix-frames
-      so that ros and opencv can operate on the camera frame correctly -->
-  <joint name="camera_optical_joint_2" type="fixed">
-    <!-- these values have to be these values otherwise the gazebo camera image
-        won't be aligned properly with the frame it is supposedly originating from -->
-    <origin xyz="0 0 0" rpy="${-pi/2} 0 ${-pi/2}"/>
-    <parent link="camera2_link"/>
-    <child link="camera_link_optical_2"/>
-  </joint>
-  <link name="camera_link_optical_2">
-  </link>
-  <!-- generate an optical frame http://www.ros.org/reps/rep-0103.html#suffix-frames
-      so that ros and opencv can operate on the camera frame correctly -->
-  <joint name="camera_optical_joint_3" type="fixed">
-    <!-- these values have to be these values otherwise the gazebo camera image
-        won't be aligned properly with the frame it is supposedly originating from -->
-    <origin xyz="0 0 0" rpy="${-pi/2} 0 ${-pi/2}"/>
-    <parent link="camera3_link"/>
-    <child link="camera_link_optical_3"/>
-  </joint>
-  <link name="camera_link_optical_3">
-</link>
   <!-- Bring in simulation data for Gazebo. -->
   <xacro:include filename="$(find ridgeback_description)/urdf/ridgeback.gazebo" />

File: ridgeback_intel_description/urdf/ridgeback_intel.urdf.xacro (robot description, xacro)
@@ -26,5 +26,5 @@
         <origin xyz="0 0 0" rpy="${PI/2} 0 0"/>
         <geometry>
-          <mesh filename="package://ridgeback_description/meshes/wheel.stl"/>
+          <mesh filename="package://ridgeback_intel_description/meshes/wheel.stl"/>
         </geometry>
         <material name="black" />
@@ -66,5 +66,5 @@
         <origin xyz="0 0 0" rpy="${PI/2} 0 ${PI/2}" />
         <geometry>
-          <mesh filename="package://ridgeback_description/meshes/rocker.stl"/>
+          <mesh filename="package://ridgeback_intel_description/meshes/rocker.stl"/>
         </geometry>
         <material name="black" />
@@ -109,5 +109,5 @@
       <origin xyz="0 0 0" rpy="0 0 0" />
       <geometry>
-        <mesh filename="package://ridgeback_description/meshes/body.stl"/>
+        <mesh filename="package://ridgeback_intel_description/meshes/body.stl"/>
       </geometry>
       <material name="black" />
@@ -116,5 +116,5 @@
       <origin xyz="0 0 0"/>
       <geometry>
-        <mesh filename="package://ridgeback_description/meshes/body-collision.stl"/>
+        <mesh filename="package://ridgeback_intel_description/meshes/body-collision.stl"/>
       </geometry>
     </collision>
@@ -142,5 +142,5 @@
       <origin xyz="0 0 0" rpy="0 0 ${PI}" />
       <geometry>
-        <mesh filename="package://ridgeback_description/meshes/side-cover.stl"/>
+        <mesh filename="package://ridgeback_intel_description/meshes/side-cover.stl"/>
       </geometry>
       <material name="yellow" />
@@ -151,5 +151,5 @@
       <origin xyz="0 0 0" rpy="0 0 0" />
       <geometry>
-        <mesh filename="package://ridgeback_description/meshes/side-cover.stl"/>
+        <mesh filename="package://ridgeback_intel_description/meshes/side-cover.stl"/>
       </geometry>
       <material name="yellow" />
@@ -165,5 +165,5 @@
       <origin xyz="0 0 0" rpy="0 0 0" />
       <geometry>
-        <mesh filename="package://ridgeback_description/meshes/end-cover.stl" />
+        <mesh filename="package://ridgeback_intel_description/meshes/end-cover.stl" />
       </geometry>
       <material name="black" />
@@ -179,5 +179,5 @@
       <origin xyz="0 0 0" rpy="0 0 ${PI}" />
       <geometry>
-        <mesh filename="package://ridgeback_description/meshes/end-cover.stl" />
+        <mesh filename="package://ridgeback_intel_description/meshes/end-cover.stl" />
       </geometry>
       <material name="black" />
@@ -198,5 +198,5 @@
       <origin xyz="0 0 0" rpy="0 0 0" />
       <geometry>
-        <mesh filename="package://ridgeback_description/meshes/lights.stl" />
+        <mesh filename="package://ridgeback_intel_description/meshes/lights.stl" />
       </geometry>
       <material name="white" />
@@ -207,5 +207,5 @@
       <origin xyz="0 0 0" rpy="0 0 ${PI}" />
       <geometry>
-        <mesh filename="package://ridgeback_description/meshes/lights.stl" />
+        <mesh filename="package://ridgeback_intel_description/meshes/lights.stl" />
       </geometry>
       <material name="red" />
@@ -221,5 +221,5 @@
       <origin xyz="0 0 0" rpy="0 0 0" />
       <geometry>
-        <mesh filename="package://ridgeback_description/meshes/top.stl" />
+        <mesh filename="package://ridgeback_intel_description/meshes/top.stl" />
       </geometry>
       <material name="black" />
@@ -228,5 +228,5 @@
       <origin xyz="0 0 0" rpy="0 0 0" />
       <geometry>
-        <mesh filename="package://ridgeback_description/meshes/top.stl"/>
+        <mesh filename="package://ridgeback_intel_description/meshes/top.stl"/>
       </geometry>
     </collision>
@@ -241,5 +241,5 @@
       <origin xyz="0 0 0" rpy="0 ${PI/2} 0" />
       <geometry>
-        <mesh filename="package://ridgeback_description/meshes/axle.stl" />
+        <mesh filename="package://ridgeback_intel_description/meshes/axle.stl" />
       </geometry>
       <material name="black" />
@@ -278,5 +278,5 @@
    <xacro:property name="angle_tilt_3" value="0" /> <!-- Space btw top of beam and the each joint -->
    <!-- Import all Gazebo-customization elements, including Gazebo colors -->
-  <xacro:include filename="$(find ridgeback_description)/urdf/multi_d435.gazebo" />
+  <xacro:include filename="$(find ridgeback_intel_description)/urdf/multi_d435.gazebo" />
   <joint name="ridgeback_to_mount" type="fixed">
     <parent link="base_link" />
@@ -295,5 +295,5 @@
           <origin xyz="0 0 0" rpy="${pi/2} 0 0"/>
           <geometry>
-    	       <mesh filename="package://ridgeback_description/meshes/tripod_simplified.STL"/>
+    	       <mesh filename="package://ridgeback_intel_description/meshes/tripod_simplified.STL"/>
           </geometry>
           <material name="orange"/>
@@ -324,5 +324,5 @@
           <origin xyz="0 0 0" rpy="0 0 ${pi/6}"/>
           <geometry>
-    	       <mesh filename="package://ridgeback_description/meshes/D435x6_mounting-support.STL"/>
+    	       <mesh filename="package://ridgeback_intel_description/meshes/D435x6_mounting-support.STL"/>
           </geometry>
         </visual>
@@ -362,5 +362,5 @@
           <origin xyz="0 0 0" rpy="${pi/2} 0 ${pi/2}"/>
           <geometry>
-    	       <mesh filename="package://ridgeback_description/meshes/Intel_RealSense_Depth_Camera_D435.STL"/>
+    	       <mesh filename="package://ridgeback_intel_description/meshes/Intel_RealSense_Depth_Camera_D435.STL"/>
           </geometry>
           <material name="red"/>
@@ -383,5 +383,5 @@
           <origin xyz="0 0 0" rpy="${pi/2} 0 ${pi/2}"/>
           <geometry>
-    	       <mesh filename="package://ridgeback_description/meshes/Intel_RealSense_Depth_Camera_D435.STL"/>
+    	       <mesh filename="package://ridgeback_intel_description/meshes/Intel_RealSense_Depth_Camera_D435.STL"/>
           </geometry>
           <material name="red"/>
@@ -404,5 +404,5 @@
           <origin xyz="0 0 0" rpy="${pi/2} 0 ${pi/2}"/>
           <geometry>
-    	       <mesh filename="package://ridgeback_description/meshes/Intel_RealSense_Depth_Camera_D435.STL"/>
+    	       <mesh filename="package://ridgeback_intel_description/meshes/Intel_RealSense_Depth_Camera_D435.STL"/>
           </geometry>
           <material name="red"/>
@@ -448,9 +448,9 @@
 </link>
   <!-- Bring in simulation data for Gazebo. -->
-  <xacro:include filename="$(find ridgeback_description)/urdf/ridgeback_intel.gazebo" />
+  <xacro:include filename="$(find ridgeback_intel_description)/urdf/ridgeback_intel.gazebo" />
   <!-- Optional standard accessories, including their simulation data. The rendering
        of these into the final description is controlled by optenv variables, which
        default each one to off.-->
-  <xacro:include filename="$(find ridgeback_description)/urdf/accessories.urdf.xacro" />
+  <xacro:include filename="$(find ridgeback_intel_description)/urdf/accessories.urdf.xacro" />
   <!-- Optional custom includes. -->
   <xacro:include filename="$(optenv RIDGEBACK_URDF_EXTRAS empty.urdf)" />
